File: Hardware/Tortoise Control Board/Tortoise Control Board.kicad_pcb (KiCad board)
At the start: 2 copper layers, 50.8 x 50.8 mm, 13 parts, among them IC1 L9110S, J1 Conn_01x02, J2 Conn_01x03, J3 Conn_01x03, J4 Conn_01x03, J5 Conn_01x08, U1 L78L09, U2 74AHC1G04GW

Commit message: Cleanup
Parts:
- IC1: footprint Package_SO:HTSOP-8-1EP_3.9x4.9mm_P1.27mm_EP2.4x3.2mm -> Package_SO:SOIC-8_3.9x4.9mm_P1.27mm
- moved J2 0.38 mm to (164.9, 97.5)
Routing:
- net Net-(IC1-Pad1): track 32.8 -> 23.1 mm, vias 2 -> 0
Changed lines of the file:
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@@
     )
   )
-  (footprint "Package_SO:HTSOP-8-1EP_3.9x4.9mm_P1.27mm_EP2.4x3.2mm" (layer "F.Cu")
+  (footprint "Package_SO:SOIC-8_3.9x4.9mm_P1.27mm" (layer "F.Cu")
     (at 142.5 100 -90)
-    (descr "HTSOP, 8 Pin (https://media.digikey.com/pdf/Data%20Sheets/Rohm%20PDFs/BD9G341EFJ.pdf), generated with kicad-footprint-generator ipc_gullwing_generator.py")
-    (tags "HTSOP SO")
+    (descr "SOIC, 8 Pin (JEDEC MS-012AA, https://www.analog.com/media/en/package-pcb-resources/package/pkg_pdf/soic_narrow-r/r_8.pdf), generated with kicad-footprint-generator ipc_gullwing_generator.py")
+    (tags "SOIC SO")
     (property "JLCPCB" "C725793")
     (property "LCSC" "C725793")
@@
       (effects (font (size 0.98 0.98) (thickness 0.15)))
     )
+    (fp_line (start 0 2.56) (end -1.95 2.56) (layer "F.SilkS") (width 0.12))
+    (fp_line (start 0 -2.56) (end -3.45 -2.56) (layer "F.SilkS") (width 0.12))
     (fp_line (start 0 2.56) (end 1.95 2.56) (layer "F.SilkS") (width 0.12))
     (fp_line (start 0 -2.56) (end 1.95 -2.56) (layer "F.SilkS") (width 0.12))
-    (fp_line (start 0 -2.56) (end -3.45 -2.56) (layer "F.SilkS") (width 0.12))
-    (fp_line (start 0 2.56) (end -1.95 2.56) (layer "F.SilkS") (width 0.12))
+    (fp_line (start -3.7 -2.7) (end -3.7 2.7) (layer "F.CrtYd") (width 0.05))
+    (fp_line (start 3.7 -2.7) (end -3.7 -2.7) (layer "F.CrtYd") (width 0.05))
+    (fp_line (start 3.7 2.7) (end 3.7 -2.7) (layer "F.CrtYd") (width 0.05))
     (fp_line (start -3.7 2.7) (end 3.7 2.7) (layer "F.CrtYd") (width 0.05))
-    (fp_line (start -3.7 -2.7) (end -3.7 2.7) (layer "F.CrtYd") (width 0.05))
-    (fp_line (start 3.7 2.7) (end 3.7 -2.7) (layer "F.CrtYd") (width 0.05))
-    (fp_line (start 3.7 -2.7) (end -3.7 -2.7) (layer "F.CrtYd") (width 0.05))
     (fp_line (start 1.95 -2.45) (end 1.95 2.45) (layer "F.Fab") (width 0.1))
+    (fp_line (start -0.975 -2.45) (end 1.95 -2.45) (layer "F.Fab") (width 0.1))
+    (fp_line (start -1.95 2.45) (end -1.95 -1.475) (layer "F.Fab") (width 0.1))
+    (fp_line (start 1.95 2.45) (end -1.95 2.45) (layer "F.Fab") (width 0.1))
     (fp_line (start -1.95 -1.475) (end -0.975 -2.45) (layer "F.Fab") (width 0.1))
-    (fp_line (start -1.95 2.45) (end -1.95 -1.475) (layer "F.Fab") (width 0.1))
-    (fp_line (start -0.975 -2.45) (end 1.95 -2.45) (layer "F.Fab") (width 0.1))
-    (fp_line (start 1.95 2.45) (end -1.95 2.45) (layer "F.Fab") (width 0.1))
-    (pad "" smd roundrect (at 0.6 0.8 270) (size 0.97 1.29) (layers "F.Paste") (roundrect_rratio 0.25))
-    (pad "" smd roundrect (at 0.6 -0.8 270) (size 0.97 1.29) (layers "F.Paste") (roundrect_rratio 0.25))
-    (pad "" smd roundrect (at -0.6 -0.8 270) (size 0.97 1.29) (layers "F.Paste") (roundrect_rratio 0.25))
-    (pad "" smd roundrect (at -0.6 0.8 270) (size 0.97 1.29) (layers "F.Paste") (roundrect_rratio 0.25))
-    (pad "1" smd roundrect (at -2.65 -1.905 270) (size 1.6 0.6) (layers "F.Cu" "F.Paste" "F.Mask") (roundrect_rratio 0.25)
+    (pad "1" smd roundrect (at -2.475 -1.905 270) (size 1.95 0.6) (layers "F.Cu" "F.Paste" "F.Mask") (roundrect_rratio 0.25)
       (net 13 "Net-(IC1-Pad1)") (pinfunction "OA") (pintype "output"))
-    (pad "2" smd roundrect (at -2.65 -0.635 270) (size 1.6 0.6) (layers "F.Cu" "F.Paste" "F.Mask") (roundrect_rratio 0.25)
+    (pad "2" smd roundrect (at -2.475 -0.635 270) (size 1.95 0.6) (layers "F.Cu" "F.Paste" "F.Mask") (roundrect_rratio 0.25)
       (net 3 "9V") (pinfunction "VCC") (pintype "power_in"))
-    (pad "3" smd roundrect (at -2.65 0.635 270) (size 1.6 0.6) (layers "F.Cu" "F.Paste" "F.Mask") (roundrect_rratio 0.25)
+    (pad "3" smd roundrect (at -2.475 0.635 270) (size 1.95 0.6) (layers "F.Cu" "F.Paste" "F.Mask") (roundrect_rratio 0.25)
       (net 3 "9V") (pinfunction "VCC") (pintype "power_in"))
-    (pad "4" smd roundrect (at -2.65 1.905 270) (size 1.6 0.6) (layers "F.Cu" "F.Paste" "F.Mask") (roundrect_rratio 0.25)
+    (pad "4" smd roundrect (at -2.475 1.905 270) (size 1.95 0.6) (layers "F.Cu" "F.Paste" "F.Mask") (roundrect_rratio 0.25)
       (net 12 "Net-(IC1-Pad4)") (pinfunction "OB") (pintype "output"))
-    (pad "5" smd roundrect (at 2.65 1.905 270) (size 1.6 0.6) (layers "F.Cu" "F.Paste" "F.Mask") (roundrect_rratio 0.25)
+    (pad "5" smd roundrect (at 2.475 1.905 270) (size 1.95 0.6) (layers "F.Cu" "F.Paste" "F.Mask") (roundrect_rratio 0.25)
       (net 1 "GND") (pinfunction "GND") (pintype "power_in"))
-    (pad "6" smd roundrect (at 2.65 0.635 270) (size 1.6 0.6) (layers "F.Cu" "F.Paste" "F.Mask") (roundrect_rratio 0.25)
+    (pad "6" smd roundrect (at 2.475 0.635 270) (size 1.95 0.6) (layers "F.Cu" "F.Paste" "F.Mask") (roundrect_rratio 0.25)
       (net 14 "Net-(IC1-Pad6)") (pinfunction "IA") (pintype "input"))
-    (pad "7" smd roundrect (at 2.65 -0.635 270) (size 1.6 0.6) (layers "F.Cu" "F.Paste" "F.Mask") (roundrect_rratio 0.25)
+    (pad "7" smd roundrect (at 2.475 -0.635 270) (size 1.95 0.6) (layers "F.Cu" "F.Paste" "F.Mask") (roundrect_rratio 0.25)
       (net 5 "SIGNAL") (pinfunction "IB") (pintype "input"))
-    (pad "8" smd roundrect (at 2.65 -1.905 270) (size 1.6 0.6) (layers "F.Cu" "F.Paste" "F.Mask") (roundrect_rratio 0.25)
+    (pad "8" smd roundrect (at 2.475 -1.905 270) (size 1.95 0.6) (layers "F.Cu" "F.Paste" "F.Mask") (roundrect_rratio 0.25)
       (net 1 "GND") (pinfunction "GND") (pintype "power_in"))
-    (pad "9" smd rect (at 0 0 270) (size 2.4 3.2) (layers "F.Cu" "F.Mask"))
-    (model "${KICAD6_3DMODEL_DIR}/Package_SO.3dshapes/HTSOP-8-1EP_3.9x4.9mm_P1.27mm_EP2.4x3.2mm.wrl"
+    (model "${KICAD6_3DMODEL_DIR}/Package_SO.3dshapes/SOIC-8_3.9x4.9mm_P1.27mm.wrl"
       (offset (xyz 0 0 0))
       (scale (xyz 1 1 1))
@@
   )
   (footprint "Connector_PinHeader_2.54mm:PinHeader_1x03_P2.54mm_Horizontal" (layer "F.Cu")
-    (at 164.5 97.5)
+    (at 164.875 97.5)
     (descr "Through hole angled pin header, 1x03, 2.54mm pitch, 6mm pin length, single row")
     (tags "Through hole angled pin header THT 1x03 2.54mm single row")
@@
   (segment (start 143.135 95.615) (end 143.135 97.375) (width 0.5) (layer "F.Cu") (net 3))
   (segment (start 163.65 88.5) (end 157.775 88.5) (width 0.5) (layer "F.Cu") (net 3))
-  (segment (start 164.5 100.04) (end 158.59 100.04) (width 0.5) (layer "F.Cu") (net 4))
+  (segment (start 164.875 100.04) (end 158.59 100.04) (width 0.5) (layer "F.Cu") (net 4))
   (segment (start 158.59 100.04) (end 157.6 99.05) (width 0.5) (layer "F.Cu") (net 4))
   (segment (start 143.135 105.96) (end 144.175 107) (width 0.5) (layer "F.Cu") (net 5))
-  (segment (start 160.08 102.58) (end 164.5 102.58) (width 0.5) (layer "F.Cu") (net 5))
   (segment (start 158.25 102.5) (end 158.17 102.58) (width 0.5) (layer "F.Cu") (net 5))
+  (segment (start 158.17 102.58) (end 164.875 102.58) (width 0.5) (layer "F.Cu") (net 5))
   (segment (start 144.175 107) (end 148.595 102.58) (width 0.5) (layer "F.Cu") (net 5))
   (segment (start 143.135 102.625) (end 143.135 105.96) (width 0.5) (layer "F.Cu") (net 5))
   (segment (start 148.595 102.58) (end 158.17 102.58) (width 0.5) (layer "F.Cu") (net 5))
   (segment (start 158.25 100.95) (end 158.25 102.5) (width 0.5) (layer "F.Cu") (net 5))
-  (segment (start 158.17 102.58) (end 160.08 102.58) (width 0.5) (layer "F.Cu") (net 5))
   (segment (start 143 116.69) (end 143 120.5) (width 1) (layer "B.Cu") (net 6))
   (segment (start 132.25 105.94) (end 143 116.69) (width 1) (layer "B.Cu") (net 6))
@@
   (segment (start 135.64 86.14) (end 140.75 91.25) (width 0.5) (layer "F.Cu") (net 12))
   (segment (start 132.25 86.14) (end 135.64 86.14) (width 0.5) (layer "F.Cu") (net 12))
+  (segment (start 140.5 100) (end 143.5 100) (width 0.5) (layer "F.Cu") (net 13))
   (segment (start 138.25 107.86) (end 138.25 102.25) (width 0.5) (layer "F.Cu") (net 13))
-  (segment (start 138.25 102.25) (end 139.25 101.25) (width 0.5) (layer "F.Cu") (net 13))
-  (segment (start 144.5 95.75) (end 144.5 97.255) (width 0.5) (layer "F.Cu") (net 13))
   (segment (start 132.25 113.86) (end 138.25 107.86) (width 0.5) (layer "F.Cu") (net 13))
-  (segment (start 139.25 101.25) (end 139.25 92.25) (width 0.5) (layer "F.Cu") (net 13))
-  (segment (start 144.5 97.255) (end 144.405 97.35) (width 0.5) (layer "F.Cu") (net 13))
-  (via (at 139.25 92.25) (size 0.8) (drill 0.4) (layers "F.Cu" "B.Cu") (net 13))
-  (via (at 144.5 95.75) (size 0.8) (drill 0.4) (layers "F.Cu" "B.Cu") (net 13))
-  (segment (start 141 92.25) (end 139.25 92.25) (width 0.5) (layer "B.Cu") (net 13))
-  (segment (start 144.5 95.75) (end 141 92.25) (width 0.5) (layer "B.Cu") (net 13))
+  (segment (start 144.405 99.095) (end 144.405 97.525) (width 0.5) (layer "F.Cu") (net 13))
+  (segment (start 138.25 102.25) (end 140.5 100) (width 0.5) (layer "F.Cu") (net 13))
+  (segment (start 143.5 100) (end 144.405 99.095) (width 0.5) (layer "F.Cu") (net 13))
   (segment (start 146.25 108.75) (end 141 108.75) (width 0.5) (layer "F.Cu") (net 14))
   (segment (start 140 106.825) (end 140.175 107) (width 0.5) (layer "F.Cu") (net 14))
