File: Hardware/Tortoise Control Board/Tortoise Control Board.kicad_sch (KiCad schematic)
At the start: 12 parts, among them IC1 L9110S, J1 Conn_01x02, J2 Conn_01x03, J3 Conn_01x03, J4 Conn_01x03, J5 Conn_01x08, U1 L78L09, U2 74AHC1G04GW

Commit message: Cleanup
Parts:
- IC1: footprint Package_SO:HTSOP-8-1EP_3.9x4.9mm_P1.27mm_EP2.4x3.2mm -> Package_SO:SOIC-8_3.9x4.9mm_P1.27mm
Changed lines of the file:
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@@
       (effects (font (size 1.27 1.27)) (justify left bottom) hide)
     )
-    (property "Footprint" "Package_SO:HTSOP-8-1EP_3.9x4.9mm_P1.27mm_EP2.4x3.2mm" (id 2) (at 175.26 101.6 0)
+    (property "Footprint" "Package_SO:SOIC-8_3.9x4.9mm_P1.27mm" (id 2) (at 175.26 101.6 0)
       (effects (font (size 1.27 1.27)) (justify left bottom) hide)
     )
@@
     )
     (path "/cf512827-0083-476a-af94-fe5e81c9a2c2"
-      (reference "IC1") (unit 1) (value "L9110S") (footprint "Package_SO:HTSOP-8-1EP_3.9x4.9mm_P1.27mm_EP2.4x3.2mm")
+      (reference "IC1") (unit 1) (value "L9110S") (footprint "Package_SO:SOIC-8_3.9x4.9mm_P1.27mm")
     )
     (path "/2efe821f-f45d-448b-95a8-7ea0f33d2d83"
