File: Hardware/Tortoise Control/Tortoise Control.kicad_sch (KiCad schematic)
At the start: 12 parts, among them IC1 L9110S, J1 Conn_01x02, J2 Conn_01x03, J3 Conn_01x03, J4 Conn_01x03, J5 Conn_01x08, U1 L78L09, U2 74AHC1G04GW

Commit message: Cleanup
Other:
- note added: "A"
- note added: "B"
- note removed: "FROG (COM)"
- note removed: "NC"
- note removed: "NO"
- note removed: "TRACK A (NO)"
- note removed: "TRACK B (NC)"
Changed lines of the file:
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@@
     (stroke (width 0) (type default) (color 0 0 0 0))
   )
-  (text "TRACK A (NO)" (at 191.77 78.74 90)
+  (text "A" (at 191.77 78.74 90)
     (effects (font (size 1 1)) (justify left bottom))
   )
-  (text "NC" (at 200.66 104.14 0)
+  (text "B" (at 200.66 104.14 0)
     (effects (font (size 1 1)) (justify left bottom))
   )
-  (text "NO" (at 200.66 96.52 0)
+  (text "B" (at 200.66 96.52 0)
     (effects (font (size 1 1)) (justify left bottom))
   )
@@
     (effects (font (size 1 1)) (justify left bottom))
   )
-  (text "NO" (at 200.66 106.68 0)
+  (text "A" (at 200.66 106.68 0)
     (effects (font (size 1 1)) (justify left bottom))
   )
-  (text "TRACK A (NO)" (at 187.96 121.92 270)
+  (text "A" (at 187.96 121.92 270)
     (effects (font (size 1 1)) (justify right bottom))
   )
@@
     (effects (font (size 1 1)) (justify left bottom))
   )
-  (text "TRACK B (NC)" (at 193.04 121.92 270)
+  (text "B" (at 193.04 121.92 270)
     (effects (font (size 1 1)) (justify right bottom))
   )
-  (text "FROG (COM)" (at 189.23 78.74 90)
+  (text "COM" (at 189.23 78.74 90)
     (effects (font (size 1 1)) (justify left bottom))
   )
@@
     (effects (font (size 1 1)) (justify left bottom))
   )
-  (text "NC" (at 200.66 93.98 0)
+  (text "A" (at 200.66 93.98 0)
     (effects (font (size 1 1)) (justify left bottom))
   )
-  (text "FROG (COM)" (at 190.5 121.92 270)
+  (text "COM" (at 190.5 121.92 270)
     (effects (font (size 1 1)) (justify right bottom))
   )
-  (text "TRACK B (NC)" (at 186.69 78.74 90)
+  (text "B" (at 186.69 78.74 90)
     (effects (font (size 1 1)) (justify left bottom))
   )
