File: Hardware/Rail Power/Rail Power.kicad_pcb (KiCad board)
At the start: 2 copper layers, 69 x 54 mm, 44 parts, among them J1 Screw_Terminal_01x02, J10 Conn_01x04, J11 Conn_01x04, J12 Conn_01x04, J13 Conn_01x04, J2 Screw_Terminal_01x02, J3 Conn_01x06, J4 Conn_01x06, J5 Conn_01x06, J6 Conn_01x06, J7 Conn_01x06, J8 Conn_01x06, J9 Screw_Terminal_01x05, K1 SRD-12VDC-SL-C, Q1 MMBT2222A 1P, SW1 SW_Push, U1 6N137, U2 LM317AG-TN3-R

Commit message: Cleanup
Parts:
- removed A1: Arduino_Nano_v3.x, Module:Arduino_Nano
- removed A2: Arduino_UNO_R3, Module:Arduino_UNO_R3_WithMountingHoles
- removed C1, C3, C4: 100nF, Capacitor_SMD:C_0603_1608Metric
- removed C2, C5: 100uF, Capacitor_SMD:C_Elec_8x10.2
- removed D1, D2, D3, D4, D6, D7: M7, Diode_SMD:D_SMA
- removed D5: 1N4148WS, Diode_SMD:D_SOD-323
- removed D8: LED, LED_SMD:LED_0603_1608Metric
- removed G***: LOGO, A.C. Wright Logo:A.C. Wright Logo 5mm
- removed J1, J2: Screw_Terminal_01x02, TerminalBlock_Phoenix:TerminalBlock_Phoenix_PT-1,5-2-3.5-H_1x02_P3.50mm_Horizontal
- removed J10, J11, J12, J13: Conn_01x04, Connector_PinHeader_2.54mm:PinHeader_1x04_P2.54mm_Vertical
- removed J3, J4, J5, J6, J7, J8: Conn_01x06, Connector_PinHeader_2.54mm:PinHeader_1x06_P2.54mm_Vertical
- removed J9: Screw_Terminal_01x05, TerminalBlock_Phoenix:TerminalBlock_Phoenix_PT-1,5-5-3.5-H_1x05_P3.50mm_Horizontal
- removed JP1: SolderJumper_2_Open, Jumper:SolderJumper-2_P1.3mm_Open_RoundedPad1.0x1.5mm
- removed K1: SRD-12VDC-SL-C, SRD-12VDC-SL-C:SRD-12VDC-SL-C
- removed Q1: MMBT2222A 1P, Package_TO_SOT_SMD:SOT-23
- removed R1, R7, R8: 1K, Resistor_SMD:R_0603_1608Metric
- removed R2, R5, R6: 10K, Resistor_SMD:R_0603_1608Metric
- removed R3: 1.5K, Resistor_SMD:R_0603_1608Metric
- removed R4: 180, Resistor_SMD:R_0603_1608Metric
- removed REF**: OSHW-Logo2_7.3x6mm_SilkScreen, Symbol:OSHW-Logo2_7.3x6mm_SilkScreen
- removed SW1: SW_Push, SW_TS-1187A-B-A-B:SW_TS-1187A-B-A-B
- removed U1: 6N137, OPTO_HCPL2630S:OPTO_HCPL2630S
- removed U2: LM317AG-TN3-R, Package_TO_SOT_SMD:TO-252-2
Routing:
- removed copper zone on B.Cu, net GND
- removed copper zone on F.Cu, net GND
Other:
- board outline removed
- board text removed: "DCC DECODER"
- board text removed: "JLCJLCJLCJLC"
- board text removed: "REV A"

Commit message: Add Rail Power
Parts:
- added C1: 100uF, Capacitor_SMD:C_Elec_8x10.2, F.Cu at (135.0, 94.5)
- added C2: 100uF, Capacitor_SMD:C_Elec_8x10.2, F.Cu at (135.0, 105.0)
- added C3: 100nF, Capacitor_SMD:C_0603_1608Metric, F.Cu at (145.2, 83.2)
- added C4: 100nF, Capacitor_SMD:C_0603_1608Metric, F.Cu at (145.5, 111.8)
- added C5: 1uF, Capacitor_Tantalum_SMD:CP_EIA-3216-18_Kemet-A, F.Cu at (148.8, 84.5)
- added C6: 1uF, Capacitor_Tantalum_SMD:CP_EIA-3216-18_Kemet-A, F.Cu at (148.8, 108.8)
- added D1: M7, Diode_SMD:D_SMA, F.Cu at (123.5, 102.0)
- added D2: M7, Diode_SMD:D_SMA, F.Cu at (123.5, 93.0)
- added D3: M7, Diode_SMD:D_SMA, F.Cu at (123.5, 106.5)
- added D4: M7, Diode_SMD:D_SMA, F.Cu at (123.5, 97.5)
- added D5: M7, Diode_SMD:D_SMA, F.Cu at (123.5, 85.5)
- added D6: M7, Diode_SMD:D_SMA, F.Cu at (123.5, 114.0)
- added D7: LED, LED_SMD:LED_0603_1608Metric, F.Cu at (154.5, 94.5)
- added D8: LED, LED_SMD:LED_0603_1608Metric, F.Cu at (154.5, 105.5)
- added H1: MountingHole, MountingHole:MountingHole_3.2mm_M3, F.Cu at (114.0, 79.0)
- added H2: MountingHole, MountingHole:MountingHole_3.2mm_M3, F.Cu at (156.0, 79.0)
- added H3: MountingHole, MountingHole:MountingHole_3.2mm_M3, F.Cu at (156.0, 121.0)
- added H4: MountingHole, MountingHole:MountingHole_3.2mm_M3, F.Cu at (114.0, 121.0)
- added J1: Screw_Terminal_01x02, TerminalBlock_Phoenix:TerminalBlock_Phoenix_PT-1,5-2-3.5-H_1x02_P3.50mm_Horizontal, F.Cu at (115.5, 98.0)
- added J2: Screw_Terminal_01x02, TerminalBlock_Phoenix:TerminalBlock_Phoenix_PT-1,5-2-3.5-H_1x02_P3.50mm_Horizontal, F.Cu at (154.3, 90.2)
- added J3: Screw_Terminal_01x02, TerminalBlock_Phoenix:TerminalBlock_Phoenix_PT-1,5-2-3.5-H_1x02_P3.50mm_Horizontal, F.Cu at (154.3, 113.5)
- added R1: 1.5K, Resistor_SMD:R_0603_1608Metric, F.Cu at (145.2, 87.8)
- added R2: 560, Resistor_SMD:R_0603_1608Metric, F.Cu at (145.5, 116.2)
- added R3: 180, Resistor_SMD:R_0603_1608Metric, F.Cu at (148.5, 90.2)
- added R4: 180, Resistor_SMD:R_0603_1608Metric, F.Cu at (148.8, 114.0)
- added R5: 1K, Resistor_SMD:R_0603_1608Metric, F.Cu at (154.5, 97.5)
- added R6: 330, Resistor_SMD:R_0603_1608Metric, F.Cu at (154.5, 102.5)
- added REF**: OSHW-Logo_5.7x6mm_SilkScreen, Symbol:OSHW-Logo_5.7x6mm_SilkScreen, F.Cu at (135.0, 121.0)
- added U1: LM317AG-TN3-R, Package_TO_SOT_SMD:TO-252-2, F.Cu at (136.8, 85.5)
- added U2: LM317AG-TN3-R, Package_TO_SOT_SMD:TO-252-2, F.Cu at (137.0, 114.0)
- added kibuzzard-620B7D00: G***, kibuzzard-620B7D00, F.Cu at (134.5, 79.0)
Routing:
- net Net-(C1-Pad1): track 0.00 -> 84.6 mm
- net Net-(C5-Pad1): track 0.00 -> 58.3 mm, vias 0 -> 2
- net Net-(C6-Pad1): track 0.00 -> 42.3 mm
- net Net-(R2-Pad2): track 0.00 -> 12.9 mm
- net Net-(D2-Pad1): track 0.00 -> 10.7 mm
- net Net-(D1-Pad1): track 0.00 -> 10.7 mm
- net Net-(R1-Pad2): track 0.00 -> 8.74 mm
- net Net-(D8-Pad2): track 0.00 -> 3.02 mm
- net Net-(D7-Pad2): track 0.00 -> 3.02 mm
- added copper zone on B.Cu, net GND
- added copper zone on F.Cu, net GND
Other:
- board outline added: 50 x 50 mm
- board text added: "12V"
- board text added: "5V"
- board text added: "GND"
- board text added: "REV A"
- board text added: "TRACK"
- board text added: "© 2022 WRIGHT TRAIN WORKS"
