File: Hardware/DCC Decoder Shield/DCC Decoder Shield.kicad_pcb (KiCad board)
At the start: 2 copper layers, 69 x 54 mm, 44 parts, among them J1 Screw_Terminal_01x02, J10 Conn_01x04, J11 Conn_01x04, J12 Conn_01x04, J13 Conn_01x04, J2 Screw_Terminal_01x02, J3 Conn_01x06, J4 Conn_01x06, J5 Conn_01x06, J6 Conn_01x06, J7 Conn_01x06, J8 Conn_01x06, J9 Screw_Terminal_01x05, K1 SRD-12VDC-SL-C, Q1 MMBT2222A 1P, SW1 SW_Push, U1 6N137, U2 LM317AG-TN3-R

Commit message: Cleanup
Parts:
- removed C2, C5: 100uF, Capacitor_SMD:C_Elec_8x10.2
- removed C3, C4: 100nF, Capacitor_SMD:C_0603_1608Metric
- removed D3, D4, D6, D7: M7, Diode_SMD:D_SMA
- removed D5: 1N4148WS, Diode_SMD:D_SOD-323
- removed D8: LED, LED_SMD:LED_0603_1608Metric
- removed G***: LOGO, A.C. Wright Logo:A.C. Wright Logo 5mm
- removed JP1: SolderJumper_2_Open, Jumper:SolderJumper-2_P1.3mm_Open_RoundedPad1.0x1.5mm
- removed R6: 10K, Resistor_SMD:R_0603_1608Metric
- removed R7, R8: 1K, Resistor_SMD:R_0603_1608Metric
- removed REF**: OSHW-Logo2_7.3x6mm_SilkScreen, Symbol:OSHW-Logo2_7.3x6mm_SilkScreen
- removed U2: LM317AG-TN3-R, Package_TO_SOT_SMD:TO-252-2
- A1: value Arduino_Nano_v3.x -> Arduino_UNO_R3; footprint Module:Arduino_Nano -> Module:Arduino_UNO_R3_WithMountingHoles
- A2: value Arduino_UNO_R3 -> Arduino_Nano_v3.x; footprint Module:Arduino_UNO_R3_WithMountingHoles -> Module:Arduino_Nano
- D1: value M7 -> 1N4148WS; footprint Diode_SMD:D_SMA -> Diode_SMD:D_SOD-323
- J13: value Conn_01x04 -> Screw_Terminal_01x05; footprint Connector_PinHeader_2.54mm:PinHeader_1x04_P2.54mm_Vertical -> TerminalBlock_Phoenix:TerminalBlock_Phoenix_PT-1,5-5-3.5-H_1x05_P3.50mm_Horizontal
- J9: value Screw_Terminal_01x05 -> Conn_01x04; footprint TerminalBlock_Phoenix:TerminalBlock_Phoenix_PT-1,5-5-3.5-H_1x05_P3.50mm_Horizontal -> Connector_PinHeader_2.54mm:PinHeader_1x04_P2.54mm_Vertical
- K1: value SRD-12VDC-SL-C -> SRD-5VDC-SL-C; footprint SRD-12VDC-SL-C:SRD-12VDC-SL-C -> SRD-5VDC-SL-C:SRD-5VDC-SL-C
- R3: value 1.5K -> 10K
- R4: value 180 -> 10K
- R5: value 10K -> 1K
- moved J10 109.1 mm to (206.8, 72.5), turned to 0 degrees
- moved D2 94.5 mm to (199.4, 102.0)
- moved J1 88.0 mm to (170.6, 127.8), turned to 0 degrees
- moved R3 87.5 mm to (210.9, 83.7)
- moved D1 87.4 mm to (179.0, 125.2)
- moved R4 62.6 mm to (124.7, 142.0)
- moved J11 61.3 mm to (211.5, 72.5), turned to 0 degrees
- moved U1 57.9 mm to (161.8, 129.3), turned to 0 degrees
- moved K1 56.1 mm to (121.6, 132.2)
- moved J6 56.1 mm to (138.9, 126.0), turned to 0 degrees
- moved J5 52.1 mm to (143.6, 126.0)
- moved J3 52.0 mm to (148.2, 126.0)
- moved J8 51.9 mm to (134.3, 126.0), turned to 0 degrees
- moved R2 48.5 mm to (120.7, 142.0), turned to 0 degrees
- moved J4 47.2 mm to (184.8, 71.3)
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Connections:
- A1 pad 1: D1 -> unconnected-(A1-Pad1)
- A1 pad 10: D7 -> A1
- A1 pad 11: D8 -> A2
- A1 pad 12: TURNOUT C -> A3
- A1 pad 13: TURNOUT D -> A4
- A1 pad 14: D11 -> A5
- A1 pad 15: D12 -> D0
- A1 pad 16: D13 -> D1
- A1 pad 17: 3V3 -> DCC
- A1 pad 18: AREF -> LEARN
- A1 pad 19: A0 -> LIGHTS
- A1 pad 2: D0 -> unconnected-(A1-Pad2)
- A1 pad 20: A1 -> TURNOUT A
- A1 pad 21: A2 -> TURNOUT B
- A1 pad 22: A3 -> D7
- A1 pad 23: A4 -> D8
- A1 pad 24: A5 -> TURNOUT C
- A1 pad 25: unconnected-(A1-Pad25) -> TURNOUT D
- A1 pad 26: unconnected-(A1-Pad26) -> D11
- A1 pad 27: 5V -> D12
- A1 pad 28: ~{RESET} -> D13
- A1 pad 30: 12V -> AREF
- A1 pad 4: GND -> 3V3
- A1 pad 5: DCC -> 5V
- A1 pad 6: LEARN -> GND
- A1 pad 7: LIGHTS -> GND
- A1 pad 8: TURNOUT A -> 12V
- A1 pad 9: TURNOUT B -> A0
- A2 pad 1: unconnected-(A2-Pad1) -> D1
- A2 pad 10: A1 -> D7
- A2 pad 11: A2 -> D8
- A2 pad 12: A3 -> TURNOUT C
- A2 pad 13: A4 -> TURNOUT D
- A2 pad 14: A5 -> D11
- A2 pad 15: D0 -> D12
- A2 pad 16: D1 -> D13
- A2 pad 17: DCC -> 3V3
- A2 pad 18: LEARN -> AREF
- A2 pad 19: LIGHTS -> A0
- A2 pad 2: IOREF -> D0
- A2 pad 20: TURNOUT A -> A1
- A2 pad 21: TURNOUT B -> A2
- A2 pad 22: D7 -> A3
- A2 pad 23: D8 -> A4
- A2 pad 24: TURNOUT C -> A5
- A2 pad 25: TURNOUT D -> unconnected-(A2-Pad25)
- A2 pad 26: D11 -> unconnected-(A2-Pad26)
- A2 pad 27: D12 -> 5V
- A2 pad 28: D13 -> ~{RESET}
- A2 pad 30: AREF -> 12V
- A2 pad 4: 3V3 -> GND
- A2 pad 5: 5V -> DCC
- A2 pad 6: GND -> LEARN
- A2 pad 7: GND -> LIGHTS
- A2 pad 8: 12V -> TURNOUT A
- A2 pad 9: A0 -> TURNOUT B
- C1 pad 2: RAIL B -> Net-(C1-Pad2)
- D1 pad 1: RAIL A -> Net-(C1-Pad1)
- D1 pad 2: GND -> Net-(C1-Pad2)
- D2 pad 1: RAIL B -> 5V
- D2 pad 2: GND -> Net-(D2-Pad2)
- J1 pad 1: RAIL B -> GND
- J1 pad 2: RAIL A -> 12V
- J10 pad 2: D8 -> 5V
- J10 pad 3: D7 -> 5V
- J10 pad 4: GND -> 5V
- J11 pad 1: TURNOUT A -> GND
- J11 pad 2: TURNOUT B -> GND
- J11 pad 3: TURNOUT C -> GND
- J11 pad 4: TURNOUT D -> GND
- J12 pad 2: 5V -> D8
- J12 pad 3: 5V -> D7
- J12 pad 4: 5V -> GND
- J13 pad 1: GND -> 12V
- J13 pad 2: GND -> Net-(J13-Pad2)
- J13 pad 3: GND -> Net-(J13-Pad3)
- J13 pad 4: GND -> Net-(J13-Pad4)
- J2 pad 1: GND -> Net-(C1-Pad2)
- J2 pad 2: 12V -> Net-(J2-Pad2)
- J3 pad 1: D0 -> A0
- J3 pad 2: D1 -> A1
- J3 pad 3: D7 -> A2
- J3 pad 4: D8 -> A3
- J3 pad 5: D11 -> A4
- J3 pad 6: D12 -> A5
- J6 pad 1: A0 -> D0
- J6 pad 2: A1 -> D1
- J6 pad 3: A2 -> D7
- J6 pad 4: A3 -> D8
- J6 pad 5: A4 -> D11
- J6 pad 6: A5 -> D12
- J9 pad 1: 12V -> TURNOUT A
- J9 pad 2: Net-(J9-Pad2) -> TURNOUT B
- J9 pad 3: Net-(J9-Pad3) -> TURNOUT C
- J9 pad 4: Net-(J9-Pad4) -> TURNOUT D
- K1 pad A1: 12V -> 5V
- K1 pad A2: Net-(D7-Pad2) -> Net-(D2-Pad2)
- K1 pad COM: Net-(J9-Pad3) -> Net-(J13-Pad3)
- K1 pad NC: Net-(J9-Pad4) -> Net-(J13-Pad4)
- K1 pad NO: Net-(J9-Pad2) -> Net-(J13-Pad2)
- Q1 pad 1: Net-(D7-Pad2) -> Net-(D2-Pad2)
- R1 pad 1: RAIL A -> Net-(J2-Pad2)
- R3 pad 1: GND -> Net-(R3-Pad1)
- R3 pad 2: Net-(R3-Pad2) -> 5V
- R4 pad 1: Net-(R3-Pad2) -> DCC
- R4 pad 2: Net-(C4-Pad1) -> 5V
- R5 pad 1: Net-(R5-Pad1) -> LIGHTS
- R5 pad 2: 5V -> Net-(Q1-Pad2)
- U1 pad 3: RAIL B -> Net-(C1-Pad2)
- U1 pad 7: Net-(R5-Pad1) -> Net-(R3-Pad1)
Other:
- board size 69 x 54 mm -> 68.6 x 53.3 mm
- board text removed: "DCC DECODER"
- board text removed: "JLCJLCJLCJLC"
- board text removed: "REV A"

Commit message: More PCBs
Parts:
- removed A1: Arduino_UNO_R3, Module:Arduino_UNO_R3_WithMountingHoles
- removed A2: Arduino_Nano_v3.x, Module:Arduino_Nano
- removed J10, J11, J9: Conn_01x04, Connector_PinHeader_2.54mm:PinHeader_1x04_P2.54mm_Vertical
- removed J3, J4, J5, J6, J7, J8: Conn_01x06, Connector_PinHeader_2.54mm:PinHeader_1x06_P2.54mm_Vertical
- added D3: M7, Diode_SMD:D_SMA, F.Cu at (116.0, 87.3)
- added G: Conn_01x06, Connector_PinHeader_2.54mm:PinHeader_1x06_P2.54mm_Vertical, F.Cu at (152.0, 76.3)
- added G: Conn_01x06, Connector_PinHeader_2.54mm:PinHeader_1x06_P2.54mm_Vertical, F.Cu at (139.3, 103.3)
- added G: Conn_01x04, Connector_PinHeader_2.54mm:PinHeader_1x04_P2.54mm_Vertical, F.Cu at (133.0, 76.3)
- added R6: 1K, Resistor_SMD:R_0603_1608Metric, F.Cu at (121.0, 87.3)
- added REF**: OSHW-Logo2_7.3x6mm_SilkScreen, Symbol:OSHW-Logo2_7.3x6mm_SilkScreen, F.Cu at (112.0, 96.8)
- added S: Conn_01x04, Connector_PinHeader_2.54mm:PinHeader_1x04_P2.54mm_Vertical, F.Cu at (133.0, 71.3)
- added S: Conn_01x06, Connector_PinHeader_2.54mm:PinHeader_1x06_P2.54mm_Vertical, F.Cu at (139.3, 108.4)
- added S: Conn_01x06, Connector_PinHeader_2.54mm:PinHeader_1x06_P2.54mm_Vertical, F.Cu at (152.0, 71.3)
- added V: Conn_01x06, Connector_PinHeader_2.54mm:PinHeader_1x06_P2.54mm_Vertical, F.Cu at (139.3, 105.9)
- added V: Conn_01x04, Connector_PinHeader_2.54mm:PinHeader_1x04_P2.54mm_Vertical, F.Cu at (133.0, 73.8)
- added V: Conn_01x06, Connector_PinHeader_2.54mm:PinHeader_1x06_P2.54mm_Vertical, F.Cu at (152.0, 73.8)
- added XA1: Arduino_Uno_Shield_WTW, Arduino:Arduino_Uno_Shield_WTW, F.Cu at (102.5, 117.3)
- added kibuzzard-620C99F3: G***, kibuzzard-620C99F3, B.Cu at (123.5, 105.8)
- D2: value M7 -> LEARN; footprint Diode_SMD:D_SMA -> LED_SMD:LED_0603_1608Metric
- R5: value 1K -> 330
- moved D2 96.6 mm to (107.0, 73.8), turned to 180 degrees
- moved J2 95.5 mm to (107.5, 85.3), turned to -90 degrees
- moved J12 91.1 mm to (107.0, 79.8), turned to 90 degrees
- moved R3 81.2 mm to (133.5, 108.3), turned to -90 degrees
- moved SW1 80.1 mm to (114.0, 72.3), turned to 90 degrees
- moved R5 74.4 mm to (107.0, 70.8)
- moved R2 72.0 mm to (120.0, 70.0), turned to -90 degrees
- moved J1 67.4 mm to (107.5, 104.3), turned to -90 degrees
- moved D1 66.1 mm to (116.0, 105.3), turned to -90 degrees
- moved Q1 62.6 mm to (120.5, 94.3), turned to 180 degrees
- moved K1 44.7 mm to (134.0, 89.3)
- moved J13 44.5 mm to (152.3, 96.4), turned to 90 degrees
- moved R1 43.3 mm to (116.0, 98.8), turned to -90 degrees
- moved U1 43.1 mm to (126.0, 105.3)
- moved R4 40.2 mm to (133.5, 102.8), turned to 90 degrees
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Connections:
- D2 pad 1: 5V -> GND
- K1 pad A2: Net-(D2-Pad2) -> Net-(D3-Pad2)
- Q1 pad 1: Net-(D2-Pad2) -> Net-(D3-Pad2)
- R5 pad 1: LIGHTS -> Net-(D2-Pad2)
- R5 pad 2: Net-(Q1-Pad2) -> D13
Routing:
- net 5V: track 0.00 -> 130.6 mm
- net DCC: track 0.00 -> 73.7 mm, vias 0 -> 3
- net 12V: track 0.00 -> 61.4 mm
- net LIGHTS: track 0.00 -> 52.7 mm, vias 0 -> 2
- net D7: track 0.00 -> 50.3 mm, vias 0 -> 3
- net D8: track 0.00 -> 48.3 mm, vias 0 -> 3
- net LEARN: track 0.00 -> 43.5 mm, vias 0 -> 2
- net Net-(C1-Pad2): track 0.00 -> 33.5 mm
- net Net-(J13-Pad3): track 0.00 -> 26.4 mm
- net D11: track 0.00 -> 24.7 mm, vias 0 -> 2
- net D12: track 0.00 -> 23.7 mm, vias 0 -> 2
- net Net-(D3-Pad2): track 0.00 -> 17.3 mm
- net Net-(R3-Pad1): track 0.00 -> 16.0 mm
- net Net-(J13-Pad4): track 0.00 -> 13.3 mm
- net Net-(J13-Pad2): track 0.00 -> 13.2 mm
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Other:
- board size 68.6 x 53.3 mm -> 55 x 55 mm
- board text added: "+12V"
- board text added: "12V"
- board text added: "5V"
- board text added: "COM"
- board text added: "GND"
- board text added: "INPUTS"
- board text added: "JLCJLCJLCJLC"
- board text added: "LEARN"
- board text added: "LOCONET EXP"
- board text added: "NC"
- board text added: "NO"
- board text added: "OUTPUTS"
- board text added: "REV A"
- board text added: "SERVOS"
- board text added: "TRACK"
- board text added: "© 2022 WRIGHT TRAIN WORKS"
