File: Hardware/DCC Decoder Shield/DCC Decoder Shield.kicad_sch (KiCad schematic)
At the start: 27 parts, among them J1 Screw_Terminal_01x02, J10 Conn_01x04, J11 Conn_01x04, J12 Conn_01x04, J13 Screw_Terminal_01x05, J2 Screw_Terminal_01x02, J3 Conn_01x06, J4 Conn_01x06, J5 Conn_01x06, J6 Conn_01x06, J7 Conn_01x06, J8 Conn_01x06, J9 Conn_01x04, K1 SRD-5VDC-SL-C, Q1 MMBT2222A 1P, SW1 SW_Push, U1 6N137

Commit message: More PCBs
Parts:
- removed A1: Arduino_UNO_R3, Module:Arduino_UNO_R3_WithMountingHoles, symbol MCU_Module:Arduino_UNO_R3
- removed A2: Arduino_Nano_v3.x, Module:Arduino_Nano, symbol MCU_Module:Arduino_Nano_v3.x
- added D2: LEARN, LED_SMD:LED_0603_1608Metric, symbol Device:LED
- added R5: 330, Resistor_SMD:R_0603_1608Metric, symbol Device:R
- added XA1: Arduino_Uno_Shield_WTW, Arduino:Arduino_Uno_Shield_WTW, symbol Arduino:Arduino_Uno_Shield_WTW
- renumbered D2 to D3, R5 to R6
Connections:
- net 12V: now also XA1.VIN
- net 5V: now also XA1.5V1 (5V)
- net A0: now also XA1.A0
- net A1: now also XA1.A1
- net A2: now also XA1.A2
- net A3: now also XA1.A3
- net A4: now also XA1.A4
- net A5: now also XA1.A5
- net D0: now also XA1.D0 (D0_RX0)
- net D1: now also XA1.D1 (D1_TX0)
- net D11: now also XA1.D11
- net D12: now also XA1.D12
- net D13: now also R5.2, XA1.D13
- net D7: now also XA1.D7
- net D8: now also XA1.D8
- net DCC: now also XA1.D2 (D2_INT0)
- net GND: now also D2.1 (K), XA1.GND1 (GND), XA1.GND2 (GND), XA1.GND3 (GND)
- net LEARN: now also XA1.D3 (D3_INT1)
- net LIGHTS: now also XA1.D4
- net TURNOUT A: now also XA1.D5
- net TURNOUT B: now also XA1.D6
- net TURNOUT C: now also XA1.D9
- net TURNOUT D: now also XA1.D10 (D10_CS)
- new net: D2.2 (A), R5.1
- no-connect marks 3 -> 6
