File: Hardware/LocoNet Interface/LocoNet Interface.kicad_pcb (KiCad board)
At the start: 2 copper layers, 50 x 50 mm, 32 parts, among them J1 12V, J2 RJ12, J3 RJ12, J4 LocoNet Termination, J5 LocoNet Interface, Q1 MMBT2222A 1P, Q2 MMBT2222A 1P, Q3 MMBT2222A 1P, U1 LM393

Commit message: Cleanup
Parts:
- removed kibuzzard-620B3784: G***, kibuzzard-620B3784
- added kibuzzard-620B5DD9: G***, kibuzzard-620B5DD9, F.Cu at (135.0, 79.0)
Other:
- board text added: "REV A"

Commit message: Add Rail Power
Other:
- board text added: "+12V"
Changed lines of the file:
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@@
     (effects (font (size 1 1) (thickness 0.15)) (justify mirror))
   )
-  (gr_text "12V" (at 150.5 120) (layer "F.SilkS")
+  (gr_text "+12V" (at 150.5 120) (layer "F.SilkS")
     (effects (font (size 1 1) (thickness 0.15)))
   )
