File: Hardware/Tortoise Breakout RJ-45/Tortoise Breakout RJ-45.kicad_pcb (KiCad board)
At the start: 2 copper layers, 50 x 50 mm, 5 parts, among them J1 RJ45, J2 Conn_01x03, J3 Conn_01x08

Commit message: More PCBs
Parts:
- added J4: Conn_01x03, TerminalBlock_Phoenix:TerminalBlock_Phoenix_PT-1,5-3-5.0-H_1x03_P5.00mm_Horizontal, F.Cu at (156.8, 119.5)
- moved REF** 32.8 mm to (170.4, 87.2)
- moved J2 4.25 mm to (140.8, 119.5)
Routing:
- net Net-(J1-Pad7): track 42.0 -> 65.3 mm, vias 2 -> 3
- net Net-(J1-Pad5): track 30.0 -> 50.6 mm
- net Net-(J1-Pad6): track 34.2 -> 53.2 mm, vias 2 -> 4
- net Net-(J1-Pad4): track 47.7 -> 49.4 mm
- net Net-(J1-Pad3): track 54.2 -> 55.5 mm
- net Net-(J1-Pad2): track 55.5 -> 56.7 mm
- net Net-(J1-Pad1): track 46.7 -> 46.2 mm
